File: kicad/Visual ADC Relay Block/Visual ADC Relay Block.kicad_pcb (KiCad board)
At the start: 4 copper layers, 44.4 x 29.2 mm, 21 parts, among them J1 Conn_01x02, J2 Output1, J3 Conn_01x03, J4 Conn_01x02, J5 Output2, K1 DIPxx-1Cxx-51x, Q1 MOSFET_N, Q2 MOSFET_N

Commit message: before changing to ribbons
Parts:
- removed Q2: MOSFET_N, My Libraries:DIP-4_W7.62mm_LongPads_for_IRLD110
- added C1: 1uF, Capacitor_SMD:C_0805_2012Metric_Pad1.18x1.45mm_HandSolder, F.Cu at (163.1, 105.4)
- added C2: 1uF, Capacitor_SMD:C_0805_2012Metric_Pad1.18x1.45mm_HandSolder, F.Cu at (167.6, 84.3)
- added J6: PWR Out, Connector_PinHeader_2.54mm:PinHeader_1x03_P2.54mm_Horizontal, F.Cu at (149.0, 88.0)
- added R6: R, Resistor_SMD:R_0805_2012Metric_Pad1.20x1.40mm_HandSolder, F.Cu at (167.6, 93.2)
- added R7: R, Resistor_SMD:R_0805_2012Metric_Pad1.20x1.40mm_HandSolder, F.Cu at (167.9, 105.3)
- added R8: R, Resistor_SMD:R_0805_2012Metric_Pad1.20x1.40mm_HandSolder, F.Cu at (163.1, 96.5)
- added R9: R, Resistor_SMD:R_0805_2012Metric_Pad1.20x1.40mm_HandSolder, F.Cu at (163.1, 99.5)
- added U1: 74HCT595, Package_SO:SO-16_3.9x9.9mm_P1.27mm, B.Cu at (121.2, 108.5)
- added U2: 74HC245, Package_SO:SOIC-20W_7.5x12.8mm_P1.27mm, B.Cu at (121.0, 97.9)
- J1: value Conn_01x02 -> DAC Vin
- J2: value Output1 -> DAC Vout
- J3: value Conn_01x03 -> Data In; footprint Connector_PinSocket_2.54mm:PinSocket_1x03_P2.54mm_Horizontal -> Connector_PinSocket_2.54mm:PinSocket_1x04_P2.54mm_Horizontal
- J4: value Conn_01x02 -> Data Out; footprint Connector_PinSocket_2.54mm:PinSocket_1x02_P2.54mm_Horizontal -> Connector_PinHeader_2.54mm:PinHeader_1x04_P2.54mm_Horizontal
- J5: value Output2 -> PWR In; footprint Connector_PinHeader_2.54mm:PinHeader_1x02_P2.54mm_Horizontal -> Connector_PinSocket_2.54mm:PinSocket_1x03_P2.54mm_Horizontal
- Q1: value MOSFET_N -> P-NMOS; footprint My Libraries:DIP-4_W7.62mm_LongPads_for_IRLD110 -> Package_TO_SOT_SMD:SOT-23
- R1, R2: footprint Resistor_THT:R_Axial_DIN0207_L6.3mm_D2.5mm_P7.62mm_Horizontal -> Resistor_SMD:R_0805_2012Metric_Pad1.20x1.40mm_HandSolder
- R3: footprint Resistor_SMD:R_0805_2012Metric_Pad1.15x1.40mm_HandSolder -> Resistor_SMD:R_0805_2012Metric_Pad1.20x1.40mm_HandSolder; moved to F.Cu
- R4: footprint Resistor_SMD:R_0805_2012Metric_Pad1.15x1.40mm_HandSolder -> Resistor_SMD:R_0805_2012Metric_Pad1.20x1.40mm_HandSolder
- R5: value 2R -> R; footprint Resistor_SMD:R_0805_2012Metric_Pad1.15x1.40mm_HandSolder -> Resistor_SMD:R_0805_2012Metric_Pad1.20x1.40mm_HandSolder; moved to F.Cu
- moved R5 45.7 mm to (167.6, 90.2)
- moved J1 35.4 mm to (117.0, 104.6)
- moved J4 24.6 mm to (132.5, 87.7)
- moved J3 22.7 mm to (132.5, 111.7), turned to 90 degrees
- moved R3 20.8 mm to (167.6, 87.3)
- moved Q1 18.7 mm to (167.7, 96.9), turned to 0 degrees
- moved J5 15.2 mm to (149.4, 104.1)
Connections:
- D1 pad 1: /Relay-5V -> Net-(D1-Pad1)
- D1 pad 2: Net-(D1-Pad2) -> GND
- D3 pad 2: Net-(D2-Pad2) -> Net-(D3-Pad2)
- D4 pad 2: Net-(D2-Pad2) -> Net-(D4-Pad2)
- D5 pad 2: Net-(D2-Pad2) -> Net-(D5-Pad2)
- D6 pad 2: Net-(D2-Pad2) -> Net-(D6-Pad2)
- D7 pad 2: Net-(D2-Pad2) -> Net-(D7-Pad2)
- J3 pad 1: /LEDEnable -> GND
- J3 pad 2: GND -> /LATCH
- J3 pad 3: /BitEnable -> /CLK
- J4 pad 1: /Vref -> GND
- J4 pad 2: /Relay-5V -> /LATCH
- J5 pad 1: /Vref -> GND
- J5 pad 2: /Relay-5V -> /Vref
- JP1 pad 1: GND -> /Vin
- JP1 pad 2: /Vin -> GND
- K1 pad 3: /Relay-5V -> Net-(D1-Pad1)
- K1 pad 4: Net-(D1-Pad2) -> GND
- Q1 pad 1: /Relay-5V -> Net-(Q1-Pad1)
- Q1 pad 2: Net-(Q1-Pad2) -> VCC
- Q1 pad 3: Net-(Q1-Pad3) -> Net-(D1-Pad1)
- R3 pad 1: /LEDEnable -> Net-(Q1-Pad1)
- R3 pad 2: Net-(Q1-Pad2) -> /PFET
- R4 pad 1: Net-(D2-Pad2) -> Net-(D4-Pad2)
- R4 pad 2: Net-(Q1-Pad3) -> /LED1
- R5 pad 1: /BitEnable -> Net-(D3-Pad2)
- R5 pad 2: Net-(Q2-Pad2) -> /LED3

Commit message: time to clean up
Parts:
- removed J3: Data In, Connector_PinSocket_2.54mm:PinSocket_1x04_P2.54mm_Horizontal
- removed J4: Data Out, Connector_PinHeader_2.54mm:PinHeader_1x04_P2.54mm_Horizontal
- removed J5: PWR In, Connector_PinSocket_2.54mm:PinSocket_1x03_P2.54mm_Horizontal
- removed J6: PWR Out, Connector_PinHeader_2.54mm:PinHeader_1x03_P2.54mm_Horizontal
- added C3: 22uF, Capacitor_SMD:C_0805_2012Metric_Pad1.18x1.45mm_HandSolder, B.Cu at (146.7, 108.4)
- added C4: 22uF, Capacitor_SMD:C_0805_2012Metric_Pad1.18x1.45mm_HandSolder, B.Cu at (148.9, 108.4)
- added C5: 22uF, Capacitor_SMD:C_0805_2012Metric_Pad1.18x1.45mm_HandSolder, B.Cu at (151.0, 108.4)
- added C6: 22uF, Capacitor_SMD:C_0805_2012Metric_Pad1.18x1.45mm_HandSolder, B.Cu at (148.8, 111.5)
- added JP2: Vref, Jumper:SolderJumper-2_P1.3mm_Open_TrianglePad1.0x1.5mm, B.Cu at (127.7, 90.8)
- C2, Q1, R3, R5, R6, R7, R8, R9: moved to B.Cu
- J1: value DAC Vin -> In; footprint Connector_PinSocket_2.54mm:PinSocket_1x02_P2.54mm_Horizontal -> Connector_PinHeader_2.54mm:PinHeader_2x04_P2.54mm_Vertical
- J2: value DAC Vout -> Out; footprint Connector_PinHeader_2.54mm:PinHeader_1x02_P2.54mm_Horizontal -> Connector_PinHeader_2.54mm:PinHeader_2x04_P2.54mm_Vertical
- JP1: value SolderJumper_2_Open -> First_Module
- R1, R2: footprint Resistor_SMD:R_0805_2012Metric_Pad1.20x1.40mm_HandSolder -> Resistor_THT:R_Axial_DIN0207_L6.3mm_D2.5mm_P10.16mm_Horizontal
- U1: moved to F.Cu
- moved C2 48.6 mm to (133.7, 119.2)
- moved R3 48.4 mm to (126.1, 112.2), turned to 180 degrees
- moved R5 44.4 mm to (124.8, 102.1)
- moved Q1 43.2 mm to (126.2, 109.1), turned to 90 degrees
- moved J2 40.8 mm to (147.3, 116.1), turned to 0 degrees
- moved R9 38.4 mm to (124.7, 97.8), turned to 180 degrees
- moved JP1 34.4 mm to (147.2, 90.8)
- moved C1 32.5 mm to (133.7, 119.3), turned to 180 degrees
- moved U2 27.4 mm to (137.1, 120.0), turned to 270 degrees
- moved R4 26.7 mm to (124.7, 99.8), turned to 180 degrees
- moved U1 22.7 mm to (137.1, 124.6), turned to 90 degrees
- moved R6 19.3 mm to (149.5, 99.8)
- moved R7 18.9 mm to (149.3, 102.0)
- moved J1 14.0 mm to (125.4, 115.9), turned to 0 degrees
- moved R8 13.9 mm to (149.3, 97.7)
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Connections:
- J1 pad 1: /Vin -> /LATCH
- J1 pad 2: GND -> /CLK
- J2 pad 1: /Vout -> /LATCH
- J2 pad 2: GND -> /CLK
Other:
- board size 44.4 x 29.2 mm -> 33 x 40.6 mm
- board text removed: "Could J3 be a ribbon cable connector?"

Commit message: why won't you stop
Parts:
- added H1: MountingHole, MountingHole:MountingHole_2.7mm, F.Cu at (119.4, 86.9)
- added H2: MountingHole, MountingHole:MountingHole_2.7mm, F.Cu at (155.0, 129.7)
- added H3: MountingHole, MountingHole:MountingHole_2.7mm, F.Cu at (155.3, 86.8)
- added H4: MountingHole, MountingHole:MountingHole_2.7mm, F.Cu at (119.4, 129.7)
- JP1, JP2: moved to F.Cu
- moved JP2 29.2 mm to (137.6, 118.2)
- moved JP1 27.9 mm to (141.9, 118.2)
- moved J1 2.71 mm to (122.7, 116.2)
- moved J2 2.26 mm to (149.5, 116.2)
- moved R7 1.57 mm to (150.8, 102.5)
- moved R2 1.52 mm to (150.8, 94.9)
- moved R8 1.52 mm to (150.8, 97.4)
- moved Q1 1.37 mm to (127.4, 108.3)
- moved R6 1.33 mm to (150.8, 100.0)
- moved R3 1.27 mm to (127.4, 112.2)
- moved C1 1.20 mm to (133.1, 118.2), turned to 0 degrees
- moved C2 1.16 mm to (133.0, 118.3)
- moved D1 1.11 mm to (132.3, 112.2)
- moved R5 0.93 mm to (124.0, 102.5), turned to 180 degrees
- moved R9 0.86 mm to (124.0, 97.4)
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Other:
- board size 33 x 40.6 mm -> 43.2 x 50.2 mm
- board text removed: "move diode to inside of relay perimeter"

Commit message: Passed DRC and No Rats
Parts:
- J1: value In -> Out
- J2: value Out -> In
- moved J1 26.8 mm to (149.5, 116.2)
- moved J2 26.8 mm to (122.7, 116.2)
- moved JP1 20.1 mm to (123.8, 109.5), turned to 90 degrees
- moved C2 6.67 mm to (136.4, 112.5)
- moved H4 4.45 mm to (123.8, 129.7)
- moved H1 4.40 mm to (123.8, 86.9)
- moved H3 4.40 mm to (150.9, 86.8)
- moved H2 4.09 mm to (150.9, 129.7)
- turned C6 to 180 degrees
Connections:
- net Net-(D2-Pad2) renamed /CL6
- net Net-(D3-Pad2) renamed /CL1
- net Net-(D4-Pad2) renamed /CL2
- net Net-(D5-Pad2) renamed /CL3
- net Net-(D6-Pad2) renamed /CL4
- net Net-(D7-Pad2) renamed /CL5
- J1 pad 6: /VOut -> /Vout
- R4 pad 2: /LED1 -> /LED2
- R5 pad 2: /LED3 -> /LED1
- R7 pad 2: /LED2 -> /LED6
- R9 pad 2: /LED6 -> /LED3
Routing:
- net VCC: track 0.00 -> 100.9 mm, vias 0 -> 9
- net /Vout: track 0.00 -> 69.7 mm
- net /Vref: track 0.00 -> 55.2 mm, vias 0 -> 1
- net GND: track 0.00 -> 53.2 mm, vias 0 -> 11
- net /LED4: track 0.00 -> 46.7 mm
- net /LED3: track 0.00 -> 43.4 mm
- net /LED5: track 0.00 -> 42.1 mm
- net /LED2: track 0.00 -> 38.6 mm
- net /LED6: track 0.00 -> 37.5 mm
- net /LATCH: track 0.00 -> 35.4 mm, vias 0 -> 1
- net /LED1: track 0.00 -> 33.6 mm
- net /CLK: track 0.00 -> 31.9 mm
- net /PFET: track 0.00 -> 25.1 mm
- net /Vin: track 0.00 -> 25.0 mm, vias 0 -> 1
- net /CL3: track 0.00 -> 22.7 mm
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- added copper zone on B.Cu, net GND
- added copper zone on F.Cu, net GND
- added copper zone on In1.Cu, net VCC
- added copper zone on In2.Cu, net VCC
Other:
- board size 43.2 x 50.2 mm -> 32.9 x 50.2 mm
- net class Default: clearance 0.2 -> 0.2032; trace_width 0.25 -> 0.2032
- net class Power added: clearance 0.2032, trace_width 0.3048, via_dia 0.8, via_drill 0.4
- rule trace_clearance: 0.2 -> 0.2032

Commit message: Silk clean up
Parts:
- moved J1 1.27 mm to (148.3, 116.2)
- moved J2 1.27 mm to (123.9, 116.2)
Routing:
- net /DataOut: track 9.92 -> 15.9 mm
- net /Vref: track 55.2 -> 52.5 mm
- net /LATCH: track 35.4 -> 32.8 mm, vias 1 -> 0
- net VCC: track 100.9 -> 98.9 mm
- net /DataIn: track 15.3 -> 13.4 mm
- net /Vout: track 69.7 -> 71.2 mm
- net /LED4: track 46.7 -> 47.6 mm
- net /LED5: track 42.1 -> 43.0 mm
- net /LED6: track 37.5 -> 38.4 mm
- net Net-(U1-Pad15): track 16.1 -> 15.5 mm
- net GND: track 53.2 -> 52.9 mm, vias 11 -> 9
Other:
- board text added: "In"
- board text added: "Out"
- board text added: "Vin"
- board text added: "Vref"

Commit message: change in/out but need to save brains
Parts:
- moved J1 24.3 mm to (123.9, 116.2)
- moved J2 24.3 mm to (148.3, 116.2)
Connections:
- J2 pad 1: /LATCH -> /CLK
- J2 pad 2: /CLK -> /LATCH
- J2 pad 3: /DataIn -> GND
- J2 pad 4: GND -> /DataIn
- J2 pad 5: GND -> /Vin
- J2 pad 6: /Vin -> GND
- J2 pad 7: /Vref -> VCC
- J2 pad 8: VCC -> /Vref
Routing:
- net VCC: track 98.9 -> 88.4 mm
- net /Vref: track 52.5 -> 43.7 mm
- net /LATCH: track 32.8 -> 25.8 mm
- net /CLK: track 31.6 -> 24.7 mm
- net /DataOut: track 15.9 -> 9.52 mm
- net /Vin: track 25.4 -> 20.5 mm
- net /DataIn: track 13.4 -> 11.5 mm
- net /Vout: track 71.2 -> 69.5 mm

Commit message: pass DRC yay!
Parts:
- J2: moved to B.Cu
- moved J2 2.37 mm to (150.6, 116.2), turned to 180 degrees
Connections:
- J2 pad 1: /CLK -> /LATCH
- J2 pad 2: /LATCH -> /CLK
- J2 pad 3: GND -> /DataIn
- J2 pad 4: /DataIn -> GND
- J2 pad 5: /Vin -> GND
- J2 pad 6: GND -> /Vin
- J2 pad 7: VCC -> /Vref
- J2 pad 8: /Vref -> VCC
Routing:
- net /Vout: track 69.5 -> 117.7 mm, vias 0 -> 1
- net /Vin: track 20.5 -> 58.9 mm
- net /DataOut: track 9.52 -> 38.8 mm, vias 0 -> 3
- net /Vref: track 43.7 -> 61.6 mm
- net /LATCH: track 25.8 -> 35.0 mm
- net /DataIn: track 11.5 -> 17.8 mm, vias 0 -> 2
- net VCC: track 88.4 -> 82.2 mm
- net /CLK: track 24.7 -> 26.6 mm
