File: kicad/Visual ADC Relay Block/Visual ADC Relay Block.sch (KiCad schematic (older format))
At the start: 34 parts, among them J1 Out, J2 In, K1 DIPxx-1Cxx-51x, Q1 pmv50epear, U1 74HCT595, U2 74HC245

Commit message: stream 21-03-05
Connections:
- net Vin is gone; now on net GND: J2.6 (Pin_6), JP1.1 (A), R1.2
Changed lines of the file:
@@
 Text Notes 6500 7100 0    50   ~ 0
 Mounting Holes
+$Comp
+L power:GND #PWR?
+U 1 1 60422000
+P 5600 1750
+F 0 "#PWR?" H 5600 1500 50  0001 C CNN
+F 1 "GND" H 5605 1577 50  0000 C CNN
+F 2 "" H 5600 1750 50  0001 C CNN
+F 3 "" H 5600 1750 50  0001 C CNN
+	1    5600 1750
+	1    0    0    -1
+$EndComp
 $EndSCHEMATC
