File: kicad/Sample-Hold-Compare/Sample-Hold-Compare.sch (KiCad schematic (older format))
At the start: 12 parts, among them U1 74HCT04, U2 74HCT04, U3 74HCT04

Commit message: stream 21-03-05
Parts:
- added D?: LED_Small, symbol Device:LED_Small
- added Q?: 2N2219, Package_TO_SOT_THT:TO-39-3, symbol Transistor_BJT:2N2219
- added R?: 6.8k, symbol Device:R_Small
- added R?: 330, symbol Device:R_Small
- U1: value 74HCT04 -> LF398
- U2: value 74HCT04 -> LM358
Connections:
- net GND: now also R?.1, R?.1
- new net: D?.1 (K), R?.2
- new net +5V: D?.2 (A), R?.2
Other:
- moved on the sheet: C1, C2, C3, C4, C5, D1, R1, R2, R3, U1, U2A, U2C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
